Commit message: faet: adding imu link, joint and sensor

File: xacro/gazebo.xacro (robot description, xacro)
@@ -4,5 +4,5 @@
       <plugin name="p3d_base_controller" filename="libgazebo_ros_p3d.so">
         <ros>
-            <argument>odom:=odom/ground_truth</argument>
+            <remapping>odom:=odom/ground_truth</remapping>
         </ros>
         <body_name>base_link</body_name>
@@ -19,23 +19,59 @@
       </plugin>
     </gazebo>
-    <!-- <gazebo reference="imu_link">
-        <gravity>true</gravity>
+    <gazebo reference="imu_link">
         <sensor name="imu_sensor" type="imu">
             <always_on>true</always_on>
-            <update_rate>1000</update_rate>
-            <visualize>true</visualize>
-            <topic>__default_topic__</topic>
-            <plugin filename="libgazebo_ros_imu_sensor.so" name="imu_plugin">
-                <topicName>trunk_imu</topicName>
-                <bodyName>imu_link</bodyName>
-                <updateRateHZ>1000.0</updateRateHZ>
-                <gaussianNoise>0.0</gaussianNoise>
-                <xyzOffset>0 0 0</xyzOffset>
-                <rpyOffset>0 0 0</rpyOffset>
-                <frameName>imu_link</frameName>
+            <update_rate>100</update_rate>
+            <imu>
+            <angular_velocity>
+                <x>
+                <noise type="gaussian">
+                    <mean>0.0</mean>
+                    <stddev>2e-4</stddev>
+                </noise>
+                </x>
+                <y>
+                <noise type="gaussian">
+                    <mean>0.0</mean>
+                    <stddev>2e-4</stddev>
+                </noise>
+                </y>
+                <z>
+                <noise type="gaussian">
+                    <mean>0.0</mean>
+                    <stddev>2e-4</stddev>
+                </noise>
+                </z>
+            </angular_velocity>
+            <linear_acceleration>
+                <x>
+                <noise type="gaussian">
+                    <mean>0.0</mean>
+                    <stddev>1.7e-2</stddev>
+                </noise>
+                </x>
+                <y>
+                <noise type="gaussian">
+                    <mean>0.0</mean>
+                    <stddev>1.7e-2</stddev>
+                </noise>
+                </y>
+                <z>
+                <noise type="gaussian">
+                    <mean>0.0</mean>
+                    <stddev>1.7e-2</stddev>
+                </noise>
+                </z>
+            </linear_acceleration>
+            </imu>
+            <plugin name="imu_plugin" filename="libgazebo_ros_imu_sensor.so">
+                <ros>
+                    <namespace>imu</namespace>
+                    <remapping>~/out:=data</remapping>
+                </ros>
+                <initial_orientation_as_reference>false</initial_orientation_as_reference>
             </plugin>
-            <pose>0 0 0 0 0 0</pose>
         </sensor>
-    </gazebo> -->
+    </gazebo>
     <!-- <gazebo reference="base_link">
         <turnGravityOff>false</turnGravityOff>

File: xacro/robot.xacro (robot description, xacro)
@@ -56,5 +56,5 @@
         </inertial>
     </link>
-    <!-- <joint name="imu_joint" type="fixed">
+    <joint name="imu_joint" type="fixed">
         <parent link="trunk"/>
         <child link="imu_link"/>
@@ -79,5 +79,5 @@
             </geometry>
         </collision>
-    </link> -->
+    </link>
     <!--
     <joint name="load_joint" type="fixed">
